Commit message: 静歩行を実装
・モデルのバグを修正(参考:chvmp/spotmicro_description)

File: spot_description/urdf/spotmicroai.urdf (robot description, URDF)
Before this commit: robot SpotMicroAI, 23 links, 22 joints
Links:
- added link base_inertia, mass 2.80; collision box size=0.14 0.11 0.07; visual mesh filename=package://spot_description/meshes/stl/mainbody.stl scale=0.001 0.001 0.001
- link base_link: mass 2.80 -> None; geometry 
- link front_left_foot_link: geometry collision box size=0.026 0.020 0.13; visual mesh filename=package://spot_description/meshes/stl/lfoot.stl scale=0.001 0.001 0.001
- link front_left_leg_link: geometry collision box size=0.028 0.036 0.109; visual mesh filename=package://spot_description/meshes/stl/larm.stl scale=0.001 0.001 0.001
- link front_left_leg_link_cover: geometry visual mesh filename=package://spot_description/meshes/stl/larm_cover.stl scale=0.001 0.001 0.001
- link front_left_shoulder_link: geometry collision box size=0.044 0.038 0.07; visual mesh filename=package://spot_description/meshes/stl/lshoulder.stl scale=0.001 0.001 0.001
- link front_left_toe_link: geometry collision sphere radius=0.02; visual mesh filename=package://spot_description/meshes/stl/foot.stl scale=0.001 0.001 0.001
- link front_link: geometry collision box size=0.058 0.11 0.07; visual mesh filename=package://spot_description/meshes/stl/frontpart.stl scale=0.001 0.001 0.001
- link front_right_foot_link: geometry collision box size=0.026 0.020 0.13; visual mesh filename=package://spot_description/meshes/stl/rfoot.stl scale=0.001 0.001 0.001
- link front_right_leg_link: geometry collision box size=0.028 0.036 0.109; visual mesh filename=package://spot_description/meshes/stl/rarm.stl scale=0.001 0.001 0.001
- link front_right_leg_link_cover: geometry visual mesh filename=package://spot_description/meshes/stl/rarm_cover.stl scale=0.001 0.001 0.001
- link front_right_shoulder_link: geometry collision box size=0.044 0.038 0.07; visual mesh filename=package://spot_description/meshes/stl/rshoulder.stl scale=0.001 0.001 0.001
- link front_right_toe_link: geometry collision sphere radius=0.02; visual mesh filename=package://spot_description/meshes/stl/foot.stl scale=0.001 0.001 0.001
- link rear_left_foot_link: geometry collision box size=0.026 0.020 0.13; visual mesh filename=package://spot_description/meshes/stl/lfoot.stl scale=0.001 0.001 0.001
- link rear_left_leg_link: geometry collision box size=0.028 0.036 0.109; visual mesh filename=package://spot_description/meshes/stl/larm.stl scale=0.001 0.001 0.001
- link rear_left_leg_link_cover: geometry visual mesh filename=package://spot_description/meshes/stl/larm_cover.stl scale=0.001 0.001 0.001
- link rear_left_shoulder_link: geometry collision box size=0.044 0.038 0.07; visual mesh filename=package://spot_description/meshes/stl/lshoulder.stl scale=0.001 0.001 0.001
- link rear_left_toe_link: geometry collision sphere radius=0.02; visual mesh filename=package://spot_description/meshes/stl/foot.stl scale=0.001 0.001 0.001
- link rear_link: geometry collision box size=0.04 0.11 0.07; visual mesh filename=package://spot_description/meshes/stl/backpart.stl scale=0.001 0.001 0.001
- link rear_right_foot_link: geometry collision box size=0.026 0.020 0.13; visual mesh filename=package://spot_description/meshes/stl/rfoot.stl scale=0.001 0.001 0.001
- link rear_right_leg_link: geometry collision box size=0.028 0.036 0.109; visual mesh filename=package://spot_description/meshes/stl/rarm.stl scale=0.001 0.001 0.001
- link rear_right_leg_link_cover: geometry visual mesh filename=package://spot_description/meshes/stl/rarm_cover.stl scale=0.001 0.001 0.001
- link rear_right_shoulder_link: geometry collision box size=0.044 0.038 0.07; visual mesh filename=package://spot_description/meshes/stl/rshoulder.stl scale=0.001 0.001 0.001
- link rear_right_toe_link: geometry collision sphere radius=0.02; visual mesh filename=package://spot_description/meshes/stl/foot.stl scale=0.001 0.001 0.001
Joints:
- added joint base_inertia_joint: type fixed, parent base_link, child base_inertia
- joint front_left_foot: origin xyz=-0.01 0 -0.12 rpy=0 0 0 -> xyz=0.014 0 -0.109 rpy=0 0 0
- joint front_left_leg: origin xyz=0 -0.052 0 rpy=0 0 0 -> xyz=0 0.055 0 rpy=0 0 0
- joint front_left_shoulder: origin xyz=-0.093 -0.036 0 rpy=0 0 0 -> xyz=0.093 0.0395 0 rpy=0 0 0
- joint front_left_toe: origin xyz=0 0 -0.115 -> xyz=0 0 -0.13
- joint front_right_foot: origin xyz=-0.01 0 -0.12 rpy=0 0 0 -> xyz=0.014 0 -0.109 rpy=0 0 0
- joint front_right_leg: origin xyz=0 0.052 0 rpy=0 0 0 -> xyz=0 -0.055 0 rpy=0 0 0
- joint front_right_shoulder: origin xyz=-0.093 0.036 0 rpy=0 0 0 -> xyz=0.093 -0.0395 0 rpy=0 0 0
- joint front_right_toe: origin xyz=0 0 -0.115 -> xyz=0 0 -0.13
- joint rear_left_foot: origin xyz=-0.01 0 -0.12 rpy=0 0 0 -> xyz=0.014 0 -0.109 rpy=0 0 0
- joint rear_left_leg: origin xyz=0 -0.052 0 rpy=0 0 0 -> xyz=0 0.055 0 rpy=0 0 0
- joint rear_left_shoulder: origin xyz=0.093 -0.036 0 rpy=0 0 0 -> xyz=-0.093 0.0395 0 rpy=0 0 0
- joint rear_left_toe: origin xyz=0 0 -0.115 -> xyz=0 0 -0.13
- joint rear_right_foot: origin xyz=-0.01 0 -0.12 rpy=0 0 0 -> xyz=0.014 0 -0.109 rpy=0 0 0
- joint rear_right_leg: origin xyz=0 0.052 0 rpy=0 0 0 -> xyz=0 -0.055 0 rpy=0 0 0
- joint rear_right_shoulder: origin xyz=0.093 0.036 0 rpy=0 0 0 -> xyz=-0.093 -0.0395 0 rpy=0 0 0
- joint rear_right_toe: origin xyz=0 0 -0.115 -> xyz=0 0 -0.13
